File: kicad/rpi_sensor_hat.sch (KiCad schematic (older format))
At the start: 1 part, among them J1 SSW-120-03-G-D

Commit message: Added STM32 microcontroller and FRAM non-volatile memory.
Parts:
- added U?: STM32L062K8Tx, Package_QFP:LQFP-32_7x7mm_P0.8mm, symbol MCU_ST_STM32L0:STM32L062K8Tx
- added U?: FM25V10-G, Package_SO:SOIC-8-1EP_3.9x4.9mm_P1.27mm_EP2.29x3mm, symbol rpi_sensor_hat:FM25V10-G
Changed lines of the file:
@@
 Text Notes 4450 2000 0    61   ~ 0
 Connector for Raspberry Pi 4 Model B
+$Comp
+L MCU_ST_STM32L0:STM32L062K8Tx U?
+U 1 1 5FE99240
+P 8200 2900
+F 0 "U?" H 8150 1811 50  0000 C CNN
+F 1 "STM32L062K8Tx" H 8150 1720 50  0000 C CNN
+F 2 "Package_QFP:LQFP-32_7x7mm_P0.8mm" H 7700 2000 50  0001 R CNN
+F 3 "http://www.st.com/st-web-ui/static/active/en/resource/technical/document/datasheet/DM00108218.pdf" H 8200 2900 50  0001 C CNN
+	1    8200 2900
+	1    0    0    -1
+$EndComp
+$Comp
+L rpi_sensor_hat:FM25V10-G U?
+U 1 1 5FEA3E28
+P 8900 950
+F 0 "U?" H 9175 965 50  0000 C CNN
+F 1 "FM25V10-G" H 9175 874 50  0000 C CNN
+F 2 "Package_SO:SOIC-8-1EP_3.9x4.9mm_P1.27mm_EP2.29x3mm" H 8900 950 50  0001 C CNN
+F 3 "https://www.cypress.com/file/41691/download" H 8900 950 50  0001 C CNN
+	1    8900 950
+	1    0    0    -1
+$EndComp
 $EndSCHEMATC

Commit message: Aded BME280 sensor.
Parts:
- added U?: BME280, rpi_sensor_hat:Pressure_Sensor_LGA-8_2.5x2.5mm_BME280, symbol dk_Humidity-Moisture-Sensors:BME280
Changed lines of the file:
@@
+	1    0    0    -1
+$EndComp
+$Comp
+L dk_Humidity-Moisture-Sensors:BME280 U?
+U 1 1 5FEAAAE6
+P 7750 4700
+F 0 "U?" H 8078 4803 60  0000 L CNN
+F 1 "BME280" H 8078 4697 60  0000 L CNN
+F 2 "rpi_sensor_hat:Pressure_Sensor_LGA-8_2.5x2.5mm_BME280" H 7950 4900 60  0001 L CNN
+F 3 "https://ae-bst.resource.bosch.com/media/_tech/media/datasheets/BST-BME280-DS002.pdf" H 7950 5000 60  0001 L CNN
+F 4 "828-1063-1-ND" H 7950 5100 60  0001 L CNN "Digi-Key_PN"
+F 5 "BME280" H 7950 5200 60  0001 L CNN "MPN"
+F 6 "Sensors, Transducers" H 7950 5300 60  0001 L CNN "Category"
+F 7 "Humidity, Moisture Sensors" H 7950 5400 60  0001 L CNN "Family"
+F 8 "https://ae-bst.resource.bosch.com/media/_tech/media/datasheets/BST-BME280-DS002.pdf" H 7950 5500 60  0001 L CNN "DK_Datasheet_Link"
+F 9 "/product-detail/en/bosch-sensortec/BME280/828-1063-1-ND/6136314" H 7950 5600 60  0001 L CNN "DK_Detail_Page"
+F 10 "SENSOR PRESSURE HUMIDITY TEMP" H 7950 5700 60  0001 L CNN "Description"
+F 11 "Bosch Sensortec" H 7950 5800 60  0001 L CNN "Manufacturer"
+F 12 "Active" H 7950 5900 60  0001 L CNN "Status"
+	1    7750 4700
 	1    0    0    -1
 $EndComp

Commit message: Added battery and power management.
Parts:
- removed U?: STM32L062K8Tx, Package_QFP:LQFP-32_7x7mm_P0.8mm, symbol MCU_ST_STM32L0:STM32L062K8Tx
- added BAT1: BS-7, rpi_sensor_hat:Battery_Holder_Coin_2032_BS-7, symbol dk_Battery-Holders-Clips-Contacts:BS-7
- added C1: 10uF, Capacitor_SMD:C_0805_2012Metric, symbol Device:C
- added C10, C11, C2, C3, C4, C5, C6, C7, C8, C9: 0.1uF, Capacitor_SMD:C_0805_2012Metric, symbol Device:C
- added D1: MBR0520LT1G, rpi_sensor_hat:SOD-123, symbol dk_Diodes-Rectifiers-Single:MBR0520LT1G
- added D2: LG_R971-KN-1, LED_SMD:LED_0805_2012Metric, symbol rpi_sensor_hat:LG_R971-KN-1
- added J2: Conn_01x03, Connector_PinHeader_2.54mm:PinHeader_1x03_P2.54mm_Vertical, symbol Connector_Generic:Conn_01x03
- added J3: Conn_01x06, Connector_PinHeader_2.54mm:PinHeader_1x06_P2.54mm_Vertical, symbol Connector_Generic:Conn_01x06
- added Q1: BSS84, Package_TO_SOT_SMD:SOT-23, symbol Transistor_FET:BSS84
- added R1: 100K, Resistor_SMD:R_0805_2012Metric, symbol Device:R
- added R10, R19, R?: 10K, Resistor_SMD:R_0805_2012Metric, symbol Device:R
- added R14, R15, R18, R20, R21, R5, R6: 100R, Resistor_SMD:R_0805_2012Metric, symbol Device:R
- added R16, R17, R3, R4: 3.9K, Resistor_SMD:R_0805_2012Metric, symbol Device:R
- added R2: 1K, Resistor_SMD:R_0805_2012Metric, symbol Device:R
- added TP1, TP10, TP11, TP12, TP3, TP4, TP5, TP6, TP7, TP8, TP9: 5016, TestPoint:TestPoint_Pad_1.0x1.0mm, symbol dk_Test-Points:5016
- added TP2: 5016, digikey-footprints:Test_Point_3.43x1.78mm, symbol dk_Test-Points:5016
- added U2: CAT24C128, Package_SO:SOIC-8_3.9x4.9mm_P1.27mm, symbol Memory_EEPROM:CAT24C128
- added U4: STM32L062K8Tx, Package_QFP:LQFP-32_7x7mm_P0.8mm, symbol rpi_sensor_hat:STM32L062K8Tx
- U3: renamed from U?; footprint Package_SO:SOIC-8-1EP_3.9x4.9mm_P1.27mm_EP2.29x3mm -> Package_SO:SOIC-8_3.9x4.9mm_P1.27mm
- gave numbers to parts that had none: 1
Connections:
- net +3V3: now also U1.6 (VDDIO), U1.8 (VDD), U3.8 (VDD), C1.1, C2.1, C3.1, C4.1, C5.1, C6.1, C7.1, C8.1, C9.1, D1.K, Q1.2 (S), R10.1, R16.1, R17.1, R?.1, TP8.1, U4.1 (VDD), U4.17 (VDD), U4.5 (VDDA); no longer J1.1 (Pin_1), J1.17 (Pin_17)
- net GND: now also U1.1 (GND), U1.7 (GND), U3.4 (VSS), BAT1.Neg, C1.2, C2.2, C3.2, C4.2, C5.2, C6.2, C7.2, C8.2, C9.2, D2.1, J2.2 (Pin_2), J3.1 (Pin_1), R1.2, TP4.1, TP5.1, U2.1 (A0), U2.2 (A1), U2.3 (A2), U2.4 (GND), U4.16 (VSS), U4.32 (VSS)
- net GPIO0_ID_SD: now also R4.2, TP3.1, U2.5 (SDA)
- net GPIO14_TXD: now also R21.1
- net GPIO15_RXD: now also R20.1
- net GPIO1_ID_SC: now also R3.2, TP6.1, U2.6 (SCL)
- net GPIO2_SDA: now also R16.2, TP11.1, U4.30 (PB7/I2C1SDA)
- net GPIO3_SCL: now also R17.2, TP12.1, U4.29 (PB6/I2C1SCL)
- net FRAM_CS: now reaches U3.1 (~CS)
- net FRAM_CS: now also R?.2, U4.10 (PA4/SPI1NSS)
- net STM32_MISO: now reaches U3.2 (MISO)
- net STM32_MISO: now also U1.5 (SDO), TP10.1, U4.12 (PA6/SPI1MISO)
- net FRAM_~WP: now reaches U3.3 (~WP)
- net FRAM_~WP: now also U4.21 (PA11)
- net STM32_MOSI: now reaches U3.5 (MOSI)
- net STM32_MOSI: now also U1.3 (SDI), TP9.1, U4.13 (PA7/SPI1MOSI)
- net STM32_SCK: now reaches U3.6 (SCK)
- net STM32_SCK: now also U1.4 (SCK), TP7.1, U4.11 (PA5/SPI1SCK)
- net FRAM_~HOLD: now reaches U3.7 (~HOLD)
- net FRAM_~HOLD: now also U4.22 (PA12)
- net SENSOR_CS: now reaches U1.2 (CSB)
- net SENSOR_CS: now also R10.2, U4.18 (PA8)
- net +5V: no longer names the net of J1.2 (Pin_2)
- net +5V: no longer J1.4 (Pin_4)
- new net: BAT1.Pos, Q1.3 (D), TP2.1
- new net: J2.3 (Pin_3), R2.2, U2.7 (WP)
- new net: D2.2, R15.2
- new net: R20.2, U4.19 (PA9/USART1TX)
- new net: R21.2, U4.20 (PA10/USART1RX)
- new net: J3.4 (Pin_4), R5.1
- new net: J3.5 (Pin_5), R6.1
- new net +3.3VP: D1.A, J1.1 (Pin_1), J1.17 (Pin_17), Q1.1 (G), R1.1, R15.1, R2.1, R3.1, R4.1, TP1.1, U2.8 (VCC)
- new net USART2RX: R5.2, U4.9 (PA3/USART2RX)
- new net USART2TX: R6.2, U4.8 (PA2/USART2TX)
- no-connect marks 0 -> 8
Other:
- note added: "3V CR2032"
- note added: "BME280 Sensor"
- note added: "BOOT0 - low for boot from flash\nHigh for bootloader"
- note added: "Battery and Power Management"
- note added: "DNP"
- note added: "Decoupling Caps"
- note added: "FRAM"
- note added: "ID EEPROM"
- note added: "Jumper\nSet 1-2 for Read Only\nSet 2-3 for Write"
- note added: "Mounting Holes"
- note added: "Revision bits"
- moved on the sheet: J1, U1, U3

Commit message: Finished schematic rev 0.
Parts:
- removed C11: 0.1uF, Capacitor_SMD:C_0805_2012Metric, symbol Device:C
- added D3, D4: LG_R971-KN-1, LED_SMD:LED_0805_2012Metric, symbol rpi_sensor_hat:LG_R971-KN-1
- added H1, H2, H3, H4: MountingHole, MountingHole:MountingHole_2.7mm_M2.5, symbol Mechanical:MountingHole
- added J4: Conn_01x03, Connector_PinHeader_2.54mm:PinHeader_1x03_P2.54mm_Vertical, symbol Connector_Generic:Conn_01x03
- added J5: Conn_02x05_Odd_Even, Connector_PinHeader_1.27mm:PinHeader_2x05_P1.27mm_Vertical_SMD, symbol Connector_Generic:Conn_02x05_Odd_Even
- added R11, R12, R13, R22, R23, R24, R8, R9: 10K, Resistor_SMD:R_0805_2012Metric, symbol Device:R
- added R25, R26: 100R, Resistor_SMD:R_0805_2012Metric, symbol Device:R
- R14: value 100R -> 10K; MPN RC0805FR-07100RL -> RC0805JR-0710KL; PLACE (none) -> STD
- R19: value 10K -> 100R; MPN RC0805JR-0710KL -> RC0805FR-07100RL
- gave numbers to parts that had none: 1
Connections:
- net GPIO27 is gone; now on net GPIO27_IRQ: J1.13 (Pin_13)
- net +3.3VP: now also R13.1, R22.1, R8.1
- net +3V3: now also J5.1 (Pin_1), R11.1, R24.1
- net GND: now also C10.2, R14.2, D3.1, D4.1, J5.3 (Pin_3), J5.5 (Pin_5), J5.9 (Pin_9), R12.2, R23.2, R9.2
- net SWCLK: now reaches R19.1
- net SWCLK: now also U4.24 (PA14/SWCLK)
- net at R19.2: now also J5.4 (Pin_4)
- net NRST: now reaches C10.1
- net NRST: now also U4.4 (NRST), J5.10 (Pin_10), R24.2
- net REV_BIT1: now reaches R14.1
- net REV_BIT1: now also U4.15 (PB1), R13.2
- net SWDIO: now reaches R18.1
- net SWDIO: now also U4.23 (PA13/SWDIO)
- net at R18.2: now also J5.2 (Pin_2)
- net REV_BIT0: now reaches U4.14 (PB0)
- net REV_BIT0: now also R8.2, R9.1
- net STM32_LED: now reaches U4.25 (PA15)
- net STM32_LED: now also R25.1
- net REV_BIT2: now reaches U4.26 (PB3)
- net REV_BIT2: now also R22.2, R23.1
- net GPIO27_IRQ: now reaches U4.27 (PB4)
- net at U4.31 (BOOT0): now also J4.2 (Pin_2)
- net GPIO17 renamed GPIO17_LED
- net GPIO17_LED: now also R26.1
- new net: J4.1 (Pin_1), R12.1
- new net: J4.3 (Pin_3), R11.2
- new net: D3.2, R25.2
- new net: D4.2, R26.2
- no-connect marks 8 -> 34
Other:
- note added: "Debug Interface"
- note added: "Hardware Revision Bits"
- note added: "LEDS"
- note added: "MCU and Interfaces"
- note added: "SWD Interface"
- note added: "Set Jumper\n1-2 for FLASH\n2-3 for BOOTLOADER"
- note removed: "BOOT0 - low for boot from flash\nHigh for bootloader"
- note removed: "Revision bits"
- moved on the sheet: BAT1, C1, C2, C3, C4, C5, C6, C7, C8, C9, D1, D2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

Commit message: Completed rev 0 of PCB layout.
Parts:
- removed TP11, TP12: 5016, TestPoint:TestPoint_Pad_1.0x1.0mm, symbol dk_Test-Points:5016
- added R27: 100R, Resistor_SMD:R_0805_2012Metric, symbol Device:R
- added R28: 10K, Resistor_SMD:R_0805_2012Metric, symbol Device:R
- BAT1, C1, C10, C2, C3, C4, C5, C6, C7, C8, C9, D1, D2, D3, D4, J1, J2, J3, J4, Q1, R1, R10, R11, R12, R15, R18, R19, R2, R20, R21, R24, R25, R26, R3, R4, R5, R6, R7, U1, U2: PLACE (none) -> STD
- H1, H2, H3, H4, TP1, TP10, TP3, TP4, TP5, TP6, TP7, TP8, TP9: PLACE (none) -> MECH
- TP2: footprint digikey-footprints:Test_Point_3.43x1.78mm -> TestPoint:TestPoint_Pad_1.0x1.0mm; PLACE (none) -> MECH
- U3: MPN (none) -> FM25V10-G; PLACE (none) -> STD
- U4: MPN (none) -> STM32L062K8T6; PLACE (none) -> STD
Connections:
- net +3.3VP: now also C3.1, U4.27 (PB4), R28.1; no longer R13.1, R22.1, R8.1
- net +3V3: now also R13.1, R22.1, R8.1; no longer C3.1
- net GND: now also R28.2
- net GPIO27_IRQ: now also R27.1; no longer U4.27 (PB4)
- net at U4.7 (PA1): now also R27.2
- no-connect marks 34 -> 33
Other:
- moved on the sheet: C3
